File: alps64.kicad_pcb (KiCad board)
At the start: 2 copper layers, 285 x 95.2 mm, 200 parts, among them J1 USB_mini_micro_B, K00 KEYSW, K00_1 KEYSW, K00_2 KEYSW, K00_3 KEYSW, K01 KEYSW, K02 KEYSW, K03 KEYSW, K04 KEYSW, K05 KEYSW, K06 KEYSW, K07 KEYSW, K10 KEYSW, K10_1 KEYSW, K10_2 KEYSW, K11 KEYSW, K12 KEYSW, K13 KEYSW, K14 KEYSW, K15 KEYSW, K16 KEYSW, K17 KEYSW, K20 KEYSW, K20_1 KEYSW, K21 KEYSW, K21_1 KEYSW, K22 KEYSW, K23 KEYSW, K23_1 KEYSW, K23_2 KEYSW, K23_3 KEYSW, K24 KEYSW, K24_1 KEYSW, K25 KEYSW, K26 KEYSW, K27 KEYSW, K27_1 KEYSW, K30 KEYSW, K30_1 KEYSW, K31 KEYSW, K31_1 KEYSW, K32 KEYSW, K32_1 KEYSW, K32_2 ALPS_SKCM, K33 KEYSW, K34 KEYSW, K35 KEYSW, K36 KEYSW, K37 KEYSW, K40 KEYSW, K40_1 KEYSW, K40_2 KEYSW, K41 KEYSW, K42 KEYSW, K43 KEYSW, K44 KEYSW, K45 KEYSW, K46 KEYSW, K47 KEYSW, K50 KEYSW, K50_1 KEYSW, K50_2 KEYSW, K51 KEYSW, K52 KEYSW, K53 KEYSW, K54 KEYSW, K55 KEYSW, K56 KEYSW, K57 KEYSW, K60 KEYSW, K60_1 KEYSW, K60_2 KEYSW, K61 KEYSW, K62 KEYSW, K63 KEYSW, K64 KEYSW, K65 KEYSW, K66 KEYSW, K67 KEYSW, K70 KEYSW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

Commit message: Add files via upload
Parts:
- removed K00_1, K00_3, K24_1: KEYSW, keyboard_parts:ALPS_SKCM_reverse_pad
- removed K00_2, K20_1, K23_1, K23_2, K27_1, K70_1: KEYSW, keyboard_parts:ALPS_SKCM
- removed P?: GND, keyboard_parts:PIN_1
- removed P?: 5V, keyboard_parts:PIN_1
- removed P?: C6, keyboard_parts:PIN_1
- removed P?: C4, keyboard_parts:PIN_1
- removed P?: C7, keyboard_parts:PIN_1
- added ?: KEYSW, keyboard_parts:ALPS_SKCM_reverse_pad, F.Cu at (109.4, 14.3)
- added ?: KEYSW, keyboard_parts:ALPS_SKCM_reverse_pad, F.Cu at (128.5, 14.3)
- added ?: KEYSW, keyboard_parts:ALPS_SKCM_reverse_pad, F.Cu at (147.5, 14.3)
- added ?: KEYSW, keyboard_parts:ALPS_SKCM_reverse_pad, F.Cu at (166.6, 14.3)
- added ?: KEYSW, keyboard_parts:ALPS_SKCM_reverse_pad, F.Cu at (185.6, 14.3)
- added ?: KEYSW, keyboard_parts:ALPS_SKCM_reverse_pad, F.Cu at (223.7, 14.3)
- added ?: KEYSW, keyboard_parts:ALPS_SKCM_reverse_pad, F.Cu at (242.8, 14.3)
- added ?: KEYSW, keyboard_parts:ALPS_SKCM, F.Cu at (14.2, 14.3)
- added ?: KEYSW, keyboard_parts:ALPS_SKCM_reverse_pad, F.Cu at (90.4, 14.3)
- added ?: KEYSW, keyboard_parts:ALPS_SKCM_reverse_pad, F.Cu at (71.3, 14.3)
- added ?: KEYSW, keyboard_parts:ALPS_SKCM, F.Cu at (271.5, 33.4)
- added ?: KEYSW, keyboard_parts:ALPS_SKCM, F.Cu at (257.2, 52.4)
- added ?: KEYSW, keyboard_parts:ALPS_SKCM, F.Cu at (266.8, 90.5)
- added ?: KEYSW, keyboard_parts:ALPS_SKCM_reverse_pad, F.Cu at (52.3, 14.3)
- added ?: KEYSW, keyboard_parts:ALPS_SKCM_reverse_pad, F.Cu at (33.2, 14.3)
- added K00: KEYSW, keyboard_parts:ALPS_SKCM_reverse_pad, F.Cu at (207.1, 90.5)
- added K06: KEYSW, keyboard_parts:ALPS_SKCM_reverse_pad, F.Cu at (204.7, 14.3)
- added K21_1: KEYSW, keyboard_parts:ALPS_SKCM, F.Cu at (250.1, 71.4)
- added K22: KEYSW, keyboard_parts:ALPS_SKCM, F.Cu at (271.5, 71.4)
- added K27: KEYSW, keyboard_parts:ALPS_SKCM, F.Cu at (73.8, 90.5)
- added K30_1: KEYSW, keyboard_parts:ALPS_SKCM, F.Cu at (16.7, 90.5)
- G***: footprint keyboard_parts:tmk_logo -> keyboard_parts:tmk2016
- moved D27 212.7 mm to (78.9, 85.6)
- moved D27 212.3 mm to (79.5, 88.8)
- moved ? 209.6 mm to (85.7, 90.5), turned to 180 degrees
- moved Poker_oval_hole 59.6 mm to (215.1, 58.1)
- moved Poker_oval_hole 42.1 mm to (72.1, 87.4)
- moved D40 27.2 mm to (27.6, 92.1)
- moved D20 26.5 mm to (259.2, 89.5)
- moved K20 23.8 mm to (252.4, 90.5)
- moved D20 23.2 mm to (253.1, 82.0)
- moved K22 21.3 mm to (271.5, 90.5)
- moved K60 19.1 mm to (166.7, 90.5)
- moved K50 17.9 mm to (53.6, 90.5)
- moved K50_1 16.7 mm to (47.6, 90.5)
- moved K10 16.7 mm to (235.7, 90.5)
- moved K10_1 16.7 mm to (238.1, 90.5)
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- renumbered K27 to ?
Routing:
- net /matrix/col6: track 448.5 -> 532.2 mm
- net /matrix/col7: track 444.8 -> 521.4 mm, vias 1 -> 6
- net /matrix/row2: track 419.6 -> 454.8 mm, vias 1 -> 5
- net /matrix/col2: track 427.8 -> 459.7 mm
- net /matrix/row4: track 204.8 -> 234.9 mm
- net /matrix/col0: track 436.1 -> 455.4 mm, vias 0 -> 2
- net /matrix/row5: track 171.2 -> 187.9 mm
- net /matrix/row3: track 311.2 -> 325.3 mm
- net Net-(D22-Pad1): track 19.7 -> 33.5 mm
- net /matrix/row0: track 270.8 -> 257.2 mm
- net Net-(D21-Pad1): track 18.8 -> 32.0 mm
- net Net-(D36-Pad1): track 17.8 -> 30.2 mm
- net /matrix/row1: track 295.6 -> 283.6 mm
- net Net-(D70-Pad1): track 36.2 -> 25.1 mm
- net Net-(D23-Pad1): track 34.6 -> 44.7 mm
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Other:
- board size 285 x 95.2 mm -> 275.7 x 95.2 mm
- net class Default: clearance 0 -> 0.254
- rule trace_clearance: 0 -> 0.254
- board text added: "(modified layout based on...) TMK64 alps tmk-kbd.com"
- board text removed: "TMK Alps64 Rev.F"
- board text removed: "tmk-kbd.com"
